File: henboard.kicad_sch (KiCad schematic)
At the start: 23 parts, among them J4 5077CR-16SMC2-BK-TR, Q1 UMH3N, U1 LDL1117S33R, U2 CP2102N-Axx-xQFN28, U3 ESP32-S3-WROOM-1, U4 USBLC6-2P6

Commit message: add libraries to henboard
Parts:
- removed U2: CP2102N-Axx-xQFN28, Package_DFN_QFN:QFN-28-1EP_5x5mm_P0.5mm_EP3.35x3.35mm, symbol Interface_USB:CP2102N-Axx-xQFN28
- removed U3: ESP32-S3-WROOM-1, RF_Module:ESP32-S3-WROOM-1, symbol Espressif:ESP32-S3-WROOM-1
- added U2: ESP32-S3-WROOM-1, symbol ESP32-S3-WROOM-1:ESP32-S3-WROOM-1
- added U3: CP2102N-Axx-xQFN28, symbol CP2102N-Axx-xQFN28:CP2102N-Axx-xQFN28
Connections:
- net +3V3: now also U2.2 (3V3), U3.6 (VDD), U3.7 (VREGIN)
- net CHIP_PU: now also U2.3 (EN)
- net DTR: now also U3.28 (DTR)
- net Earth: now also U2.1 (GND), U2.40 (GND), U2.41 (GND), U3.29 (GND), U3.3 (GND)
- net GPIO0: now also U2.27 (GPIO0/BOOT)
- net RTS: now also U3.24 (RTS)
- net TOUCH1: now also U2.39 (GPIO1/TOUCH1/ADC1_CH0)
- net TOUCH10: now also U2.18 (GPIO10/TOUCH10/ADC1_CH9/FSPICS0/FSPIIO4/SUBSPICS0)
- net TOUCH11: now also U2.19 (GPIO11/TOUCH11/ADC2_CH0/FSPID/FSPIIO5/SUBSPID)
- net TOUCH12: now also U2.20 (GPIO12/TOUCH12/ADC2_CH1/FSPICLK/FSPIIO6/SUBSPICLK)
- net TOUCH13: now also U2.21 (GPIO13/TOUCH13/ADC2_CH2/FSPIQ/FSPIIO7/SUBSPIQ)
- net TOUCH14: now also U2.22 (GPIO14/TOUCH14/ADC2_CH3/FSPIWP/FSPIDQS/SUBSPIWP)
- net TOUCH2: now also U2.38 (GPIO2/TOUCH2/ADC1_CH1)
- net TOUCH3: now also U2.15 (GPIO3/TOUCH3/ADC1_CH2)
- net TOUCH4: now also U2.4 (GPIO4/TOUCH4/ADC1_CH3)
- net TOUCH5: now also U2.5 (GPIO5/TOUCH5/ADC1_CH4)
- net TOUCH6: now also U2.6 (GPIO6/TOUCH6/ADC1_CH5)
- net TOUCH7: now also U2.7 (GPIO7/TOUCH7/ADC1_CH6)
- net TOUCH8: now also U2.12 (GPIO8/TOUCH8/ADC1_CH7/SUBSPICS1)
- net TOUCH9: now also U2.17 (GPIO9/TOUCH9/ADC1_CH8/FSPIHD/SUBSPIHD)
- net U0RXD: now also U2.36 (U0RXD/GPIO44/CLK_OUT2), U3.26 (TXD)
- net U0TXD: now also U2.37 (U0TXD/GPIO43/CLK_OUT1), U3.25 (RXD)
- net USB_DN: now also U3.5 (D-)
- net USB_DP: now also U3.4 (D+)
- net at C9.2, R6.2, R7.1: now also U3.8 (VBUS)
- net at R18.1: now also U3.9 (~{RST})
