File: henboard.kicad_sch (KiCad schematic)
At the start: 47 parts, among them J1 5077CR-16SMC2-BK-TR, J10 Conn_01x01, J11 Conn_01x01, J12 Conn_01x01, J13 Conn_01x01, J14 Conn_01x01, J15 Conn_01x01, J16 Conn_01x01, J17 Conn_01x01, J18 Conn_01x01, J19 Conn_01x01, J2 Conn_01x01, J20 Conn_01x01, J21 Conn_01x01, J3 Conn_01x01, J4 Conn_01x01, J5 Conn_01x01, J6 Conn_01x01, J7 Conn_01x01, J8 Conn_01x01, J9 Conn_01x01, Q1 UMH3N, U1 USBLC6-2P6, U2 LDL1117S33R, U3 CP2102N-Axx-xQFN28, U4 ESP32-S3-WROOM-1

Commit message: Delete all
Parts:
- removed C1, C4, C5, C7: 10uF/25V(20%), Capacitor_SMD:C_0603_1608Metric_Pad1.08x0.95mm_HandSolder, symbol Device:C
- removed C2, C3, C8: 0.1uF/50V(10%), Capacitor_SMD:C_0603_1608Metric_Pad1.08x0.95mm_HandSolder, symbol Device:C
- removed C6, C9: 1uF/16V(10%), Capacitor_SMD:C_0603_1608Metric_Pad1.08x0.95mm_HandSolder, symbol Device:C
- removed J1: 5077CR-16SMC2-BK-TR, 5077CR-16SMC2-BK-TR:5077CR-16SMC2-BK-TR, symbol 5077CR-16SMC2-BK-TR:5077CR-16SMC2-BK-TR
- removed J10, J11, J12, J13, J14, J15, J16, J17, J18, J19, J2, J20, J21, J3, J4, J5, J6, J7, J8, J9: Conn_01x01, Pad-CapacitiveTouch:Pad-CapacitiveTouch-small, symbol Connector_Generic:Conn_01x01
- removed Q1: UMH3N, Package_TO_SOT_SMD:SOT-363_SC-70-6, symbol Transistor_BJT:UMH3N
- removed R1, R2: 5.1K(1%), Resistor_SMD:R_0603_1608Metric_Pad0.98x0.95mm_HandSolder, symbol Device:R
- removed R3: 22.1K(1%), Resistor_SMD:R_0603_1608Metric_Pad0.98x0.95mm_HandSolder, symbol Device:R
- removed R4: 47.5K(1%), Resistor_SMD:R_0603_1608Metric_Pad0.98x0.95mm_HandSolder, symbol Device:R
- removed R5: 1K(1%), Resistor_SMD:R_0603_1608Metric_Pad0.98x0.95mm_HandSolder, symbol Device:R
- removed R6: 10K(1%), Resistor_SMD:R_0603_1608Metric_Pad0.98x0.95mm_HandSolder, symbol Device:R
- removed S1, S2, S3, S4, S5, S6: SKRPACE010, SKRPACE010:SKRPACE010, symbol SKRPACE010:SKRPACE010
- removed U1: USBLC6-2P6, Package_TO_SOT_SMD:SOT-666, symbol Power_Protection:USBLC6-2P6
- removed U2: LDL1117S33R, LDL1117S33R:LDL1117S33R, symbol LDL1117S33R:LDL1117S33R
- removed U3: CP2102N-Axx-xQFN28, Package_DFN_QFN:QFN-28-1EP_5x5mm_P0.5mm_EP3.35x3.35mm, symbol CP2102N-Axx-xQFN28:CP2102N-Axx-xQFN28
- removed U4: ESP32-S3-WROOM-1, RF_Module:ESP32-S3-WROOM-1, symbol ESP32-S3-WROOM-1:ESP32-S3-WROOM-1
Connections:
- no-connect marks 45 -> 0

Commit message: Finish schematic
Parts:
- added J1, J2: Conn_01x22, Connector_PinHeader_2.54mm:PinHeader_1x22_P2.54mm_Vertical, symbol Connector_Generic:Conn_01x22
- added J10, J11, J12, J13, J14, J15, J16, J17, J18, J19, J20, J3, J4, J5, J6, J7, J8, J9: Conn_01x01, Pad-CapacitiveTouch:Pad-CapacitiveTouch-small, symbol Connector_Generic:Conn_01x01
- added S1, S2, S3, S4: SKRPACE010, SKRPACE010:SKRPACE010, symbol SKRPACE010:SKRPACE010
Connections:
- new net GND: J1.22 (Pin_22), J2.1 (Pin_1), J2.21 (Pin_21), J2.22 (Pin_22), S1.4, S2.4, S3.4, S4.4
- new net SELECT1: J1.8 (Pin_8), S1.1
- new net SELECT2: J1.9 (Pin_9), S2.1
- new net SELECT3: J1.10 (Pin_10), S3.1
- new net SELECT4: J1.11 (Pin_11), S4.1
- new net TOUCH1: J2.4 (Pin_4), J5.1 (Pin_1)
- new net TOUCH10: J1.16 (Pin_16), J12.1 (Pin_1)
- new net TOUCH11: J1.17 (Pin_17), J14.1 (Pin_1), J15.1 (Pin_1)
- new net TOUCH12: J1.18 (Pin_18), J17.1 (Pin_1)
- new net TOUCH13: J1.19 (Pin_19), J20.1 (Pin_1), J4.1 (Pin_1)
- new net TOUCH14: J1.20 (Pin_20), J19.1 (Pin_1), J3.1 (Pin_1)
- new net TOUCH2: J2.5 (Pin_5), J7.1 (Pin_1)
- new net TOUCH3: J1.13 (Pin_13), J10.1 (Pin_1)
- new net TOUCH4: J1.4 (Pin_4), J11.1 (Pin_1)
- new net TOUCH5: J1.5 (Pin_5), J13.1 (Pin_1)
- new net TOUCH6: J1.6 (Pin_6), J16.1 (Pin_1)
- new net TOUCH7: J1.7 (Pin_7), J18.1 (Pin_1)
- new net TOUCH8: J1.12 (Pin_12), J6.1 (Pin_1)
- new net TOUCH9: J1.15 (Pin_15), J8.1 (Pin_1), J9.1 (Pin_1)
- no-connect marks 0 -> 30

Commit message: Finish piano
Parts:
- removed J20, J8: Conn_01x01, Pad-CapacitiveTouch:Pad-CapacitiveTouch-small, symbol Connector_Generic:Conn_01x01
- added J15, J21, J22, J9: Conn_01x01, Pad-CapacitiveTouch:Pad-CapacitiveTouch-small, symbol Connector_Generic:Conn_01x01
- renumbered J13 to J10, J16 to J11, J18 to J12, J9 to J13, J12 to J14, J15 to J16, J10 to J18, J14 to J19, J19 to J20, J7 to J6, J11 to J7, J6 to J8
Connections:
- net TOUCH11: now also J15.1 (Pin_1); no longer J19.1 (Pin_1)
- net TOUCH13: now also J19.1 (Pin_1); no longer J4.1 (Pin_1)
- net TOUCH14: no longer J3.1 (Pin_1)
- net TOUCH3: now also J3.1 (Pin_1), J21.1 (Pin_1)
- net TOUCH5: now also J9.1 (Pin_1)
- net TOUCH8: now also J4.1 (Pin_1), J22.1 (Pin_1)
Other:
- moved on the sheet: J10, J11, J12, J13, J14, J16, J17, J18, J19, J20, J5, J6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
